Commit message: Add a LiDAR link on the drone and bridge /scan from Gazebo.
This prepares the sim stack for obstacle sensing without changing motor or spawn logic.

Co-authored-by: Cursor <cursoragent@cursor.com>

File: src/drone_robot/model/robot.xacro (robot description, xacro)
@@ -21,4 +21,29 @@
     </inertial>
   </link>
+  <!-- LiDAR Link -->
+  <link name="lidar_link">
+    <visual>
+      <geometry>
+        <cylinder radius="0.03" length="0.04"/>
+      </geometry>
+      <material name="blue">
+        <color rgba="0.0 0.0 1.0 1.0"/>
+      </material>
+    </visual>
+    <collision>
+      <geometry>
+        <cylinder radius="0.03" length="0.04"/>
+      </geometry>
+    </collision>
+    <inertial>
+      <mass value="0.1"/>
+      <inertia ixx="0.0001" ixy="0.0" ixz="0.0" iyy="0.0001" iyz="0.0" izz="0.0001"/>
+    </inertial>
+  </link>
+  <joint name="lidar_joint" type="fixed">
+    <parent link="base_link"/>
+    <child link="lidar_link"/>
+    <origin xyz="0 0 0.05" rpy="0 0 0"/>
+  </joint>
   <!-- Rotor Macro (Template to avoid repeating code 4 times) -->
   <xacro:macro name="rotor" params="name x y">
